Commit message: joint controllers all work now, but need some values changing for knees and ankles so they are correct
script to disable torque on all motors (disable_torque_startup.py)

File: zeno_description/urdf/zeno_robot.urdf (robot description, URDF)
Before this commit: robot zeno, 27 links, 26 joints
Joints:
- joint l_ankle_pitch_joint: limit lower=-1.0 upper=1.0 effort=10 velocity=1.0 -> lower=-3.1415 upper=3.1415 effort=10 velocity=1.0
- joint l_ankle_roll_joint: limit lower=-1.0 upper=1.0 effort=10 velocity=1.0 -> lower=-3.1415 upper=3.1415 effort=10 velocity=1.0
- joint l_elbow_pitch_joint: limit lower=-1.0 upper=1.0 effort=10 velocity=1.0 -> lower=-3.1415 upper=3.1415 effort=10 velocity=1.0
- joint l_elbow_roll_joint: limit lower=-1.0 upper=1.0 effort=10 velocity=1.0 -> lower=-3.1415 upper=3.1415 effort=10 velocity=1.0
- joint l_hip_pitch_joint: limit lower=-1.0 upper=1.0 effort=10 velocity=1.0 -> lower=-3.1415 upper=3.1415 effort=10 velocity=1.0
- joint l_hip_roll_joint: limit lower=-1.0 upper=1.0 effort=10 velocity=1.0 -> lower=-3.1415 upper=3.1415 effort=10 velocity=1.0
- joint l_hip_yaw_joint: limit lower=-1.0 upper=1.0 effort=10 velocity=1.0 -> lower=-3.1415 upper=3.1415 effort=10 velocity=1.0
- joint l_knee_pitch_joint: limit lower=-1.0 upper=1.0 effort=10 velocity=1.0 -> lower=-3.1415 upper=3.1415 effort=10 velocity=1.0
- joint l_shoulder_pitch_joint: limit lower=-1.0 upper=1.0 effort=10 velocity=1.0 -> lower=-3.1415 upper=3.1415 effort=10 velocity=1.0
- joint l_shoulder_roll_joint: limit lower=-1.0 upper=1.0 effort=10 velocity=1.0 -> lower=-3.1415 upper=3.1415 effort=10 velocity=1.0
- joint l_wrist_roll_joint: limit lower=-1.0 upper=1.0 effort=10 velocity=1.0 -> lower=-3.1415 upper=3.1415 effort=10 velocity=1.0
- joint neck_pitch_joint: limit lower=-1.0 upper=1.0 effort=10 velocity=1.0 -> lower=-3.1415 upper=3.1415 effort=10 velocity=1.0
- joint neck_yaw_joint: limit lower=-1.0 upper=1.0 effort=10 velocity=1.0 -> lower=-3.1415 upper=3.1415 effort=10 velocity=1.0
- joint r_ankle_pitch_joint: limit lower=-1.0 upper=1.0 effort=10 velocity=1.0 -> lower=-3.1415 upper=3.1415 effort=10 velocity=1.0
- joint r_ankle_roll_joint: limit lower=-1.0 upper=1.0 effort=10 velocity=1.0 -> lower=-3.1415 upper=3.1415 effort=10 velocity=1.0
- joint r_elbow_pitch_joint: limit lower=-1.0 upper=1.0 effort=10 velocity=1.0 -> lower=-3.1415 upper=3.1415 effort=10 velocity=1.0
- joint r_elbow_roll_joint: limit lower=-1.0 upper=1.0 effort=10 velocity=1.0 -> lower=-3.1415 upper=3.1415 effort=10 velocity=1.0
- joint r_hip_pitch_joint: limit lower=-1.0 upper=1.0 effort=10 velocity=1.0 -> lower=-3.1415 upper=3.1415 effort=10 velocity=1.0
- joint r_hip_roll_joint: limit lower=-1.0 upper=1.0 effort=10 velocity=1.0 -> lower=-3.1415 upper=3.1415 effort=10 velocity=1.0
- joint r_hip_yaw_joint: limit lower=-1.0 upper=1.0 effort=10 velocity=1.0 -> lower=-3.1415 upper=3.1415 effort=10 velocity=1.0
- joint r_knee_pitch_joint: limit lower=-1.0 upper=1.0 effort=10 velocity=1.0 -> lower=-3.1415 upper=3.1415 effort=10 velocity=1.0
- joint r_shoulder_pitch_joint: limit lower=-1.0 upper=1.0 effort=10 velocity=1.0 -> lower=-3.1415 upper=3.1415 effort=10 velocity=1.0
- joint r_shoulder_roll_joint: limit lower=-1.0 upper=1.0 effort=10 velocity=1.0 -> lower=-3.1415 upper=3.1415 effort=10 velocity=1.0
- joint r_wrist_roll_joint: limit lower=-1.0 upper=1.0 effort=10 velocity=1.0 -> lower=-3.1415 upper=3.1415 effort=10 velocity=1.0
- joint torso_joint: limit lower=-1.0 upper=1.0 effort=10 velocity=1.0 -> lower=-3.1415 upper=3.1415 effort=10 velocity=1.0

Commit message: urdf fixes, going to use xacro

File: zeno_description/urdf/zeno_robot.urdf (robot description, URDF)
Before this commit: robot zeno, 27 links, 26 joints
Joints:
- joint r_ankle_pitch_joint: origin xyz=0.0 0.0 -0.6846 rpy=0 0 0 -> xyz=0.6846 0.0 0.0 rpy=0 0 0
- joint r_ankle_roll_joint: axis (none) -> 0 0 1; origin xyz=0.0 0.0 -0.4622 rpy=0 0 0 -> xyz=0.4622 0.0 0.0 rpy=0 0 0
- joint r_elbow_pitch_joint: origin xyz=0.0 0.0 -0.128 rpy=0 0 0 -> xyz=0.25 0.0 -0.1 rpy=0 0 0
- joint r_elbow_roll_joint: axis 0 0 1 -> 1 0 0; origin xyz=0.0 -0.1 -0.7 rpy=0 0 0 -> xyz=0.7 0.0 0.0 rpy=-1.5707 0 0
- joint r_hip_pitch_joint: origin xyz=0.0 0.0 -0.448 rpy=0 0 0 -> xyz=0.448 0.0 0.0 rpy=0 0 0
- joint r_hip_roll_joint: axis 1 0 0 -> 0 0 1; origin xyz=0.0 0.0 -0.148 rpy=0 0 0 -> xyz=0.148 0.0 0.0 rpy=0 0 0
- joint r_hip_yaw_joint: axis 0 0 1 -> 1 0 0; origin xyz=0.0 -.3253 -0.41 rpy=0 0 0 -> xyz=0.0 -.3253 -0.41 rpy=0 1.5707 0
- joint r_knee_pitch_joint: origin xyz=0.0 0.0 -0.7267 rpy=0 0 0 -> xyz=0.7267 0.0 0.0 rpy=0 0 0
- joint r_shoulder_pitch_joint: axis 0 1 0 -> 1 0 0; origin xyz=0.0 -0.66 0.70 rpy=0 0 0 -> xyz=0.0 -0.66 0.70 rpy=0 -0.1418 -1.5707
- joint r_shoulder_roll_joint: axis 1 0 0 -> 0 1 0; origin xyz=0.0 -0.222 0.36 rpy=0 0 0 -> xyz=0.222 0.0 0.36 rpy=0 1.5707 0
- joint r_wrist_roll_joint: axis 0 0 1 -> 1 0 0; origin xyz=0.0 0.0 -0.292 rpy=0 0 0 -> xyz=0.292 0.0 0.1 rpy=0 0 0
