Commit message: most REP-120 links added

File: zeno_description/urdf/zeno_arm.urdf.xacro (robot description, xacro)
@@ -7,4 +7,6 @@
         <link name="${prefix}_elbow_pitch_link"/>
         <link name="${prefix}_wrist_roll_link"/>
+        <link name="${prefix}_wrist"/>
+        <link name="${prefix}_gripper"/>
         <!-- Right arm joints -->
         <joint name="${prefix}_shoulder_pitch_joint" type="revolute">
@@ -18,5 +20,5 @@
             <parent link="${prefix}_shoulder_pitch_link"/>
             <child link="${prefix}_shoulder_roll_link"/>
-            <origin xyz="0.222 0.0 0.36" rpy="0 ${pi/2} 0" />
+            <origin xyz="0.222 0.0 0.36" rpy="0 ${shoulder_roll_angle} 0" />
             <axis xyz="0 1 0"/>
             <limit velocity="1.0" effort="10" lower="-3.1415" upper="3.1415" />
@@ -25,5 +27,5 @@
             <parent link="${prefix}_shoulder_roll_link"/>
             <child link="${prefix}_elbow_roll_link"/>
-            <origin xyz="0.7 0.0 0.0" rpy="${reflect * pi/2} 0 0" />
+            <origin xyz="0.7 0.0 0.0" rpy="0 0 0" />
             <axis xyz="1 0 0"/>
             <limit velocity="1.0" effort="10" lower="-3.1415" upper="3.1415" />
@@ -32,5 +34,5 @@
             <parent link="${prefix}_elbow_roll_link"/>
             <child link="${prefix}_elbow_pitch_link"/>
-            <origin xyz="0.25 0.0 -0.1" rpy="0 0 0" />
+            <origin xyz="0.25 ${reflect * 0.1} 0.0" rpy="0 0 0" />
             <axis xyz="0 1 0"/>
             <limit velocity="1.0" effort="10" lower="-3.1415" upper="3.1415" />
@@ -39,8 +41,18 @@
             <parent link="${prefix}_elbow_pitch_link"/>
             <child link="${prefix}_wrist_roll_link"/>
-            <origin xyz="0.292 0.0 0.1" rpy="0 0 0" />
+            <origin xyz="0.292 ${reflect * -0.1} 0.0" rpy="0 0 0" />
             <axis xyz="1 0 0"/>
             <limit velocity="1.0" effort="10" lower="-3.1415" upper="3.1415" />
         </joint>
+        <joint name="${prefix}_wrist_joint" type="fixed">
+            <parent link="${prefix}_wrist_roll_link"/>
+            <child link="${prefix}_wrist"/>
+            <origin xyz="0.32 0.0 0.0" rpy="0 0 0" />
+        </joint>
+        <joint name="${prefix}_gripper_joint" type="fixed">
+            <parent link="${prefix}_wrist"/>
+            <child link="${prefix}_gripper"/>
+            <origin xyz="0.5 0.0 0.0" rpy="0 0 0" />
+        </joint>
     </xacro:macro>
 </robot>

File: zeno_description/urdf/zeno_head.urdf.xacro (robot description, xacro)
@@ -5,8 +5,7 @@
         <link name="neck_yaw_link"/>
         <link name="neck_pitch_link"/>
-        <!--<link name="neck_roll_link"/>-->
-        <!--<link name="gaze_link_link"/>-->
-        <!--<link name="l_eye_gaze_link"/>-->
-        <!--<link name="r_eye_gaze_link"/>-->
+        <link name="neck_roll_link"/>
+        <link name="gaze"/>
+        <!--<link name="l_eye_camera"/>-->
         <!-- Head joints -->
         <joint name="neck_yaw_joint" type="revolute">
@@ -20,8 +19,20 @@
             <parent link="neck_yaw_link"/>
             <child link="neck_pitch_link"/>
-            <origin xyz="0.0 0.0 0.3" rpy="0 0 0" />
+            <origin xyz="0.05 0.0 0.3" rpy="0 0 0" />
             <axis xyz="0 1 0"/>
             <limit velocity="1.0" effort="10" lower="-3.1415" upper="3.1415" />
         </joint>
+        <joint name="neck_roll_joint" type="revolute">
+            <parent link="neck_pitch_link"/>
+            <child link="neck_roll_link"/>
+            <origin xyz="0.0 0.0 0.056" rpy="0 0 0" />
+            <axis xyz="1 0 0"/>
+            <limit velocity="1.0" effort="10" lower="-3.1415" upper="3.1415" />
+        </joint>
+        <joint name="gaze_joint" type="fixed">
+            <parent link="neck_roll_link"/>
+            <child link="gaze"/>
+            <origin xyz="0.55 0.0 0.55" rpy="0 0 0" />
+        </joint>
     </xacro:macro>
 </robot>

File: zeno_description/urdf/zeno_leg.urdf.xacro (robot description, xacro)
@@ -8,8 +8,10 @@
         <link name="${prefix}_ankle_pitch_link"/>
         <link name="${prefix}_ankle_roll_link"/>
+        <link name="${prefix}_sole"/>
+        <link name="${prefix}_toe"/>
         <joint name="${prefix}_hip_yaw_joint" type="revolute">
             <parent link="pelvis_link"/>
             <child link="${prefix}_hip_yaw_link"/>
-            <origin xyz="0.0 ${reflect * 0.3253}  -0.41" rpy="0 ${pi/2} 0" />
+            <origin xyz="0.15 ${reflect * 0.3253}  -0.41" rpy="0 ${pi/2} 0" />
             <axis xyz="1 0 0"/>
             <limit velocity="1.0" effort="10" lower="-3.1415" upper="3.1415" />
@@ -25,5 +27,5 @@
             <parent link="${prefix}_hip_roll_link"/>
             <child link="${prefix}_hip_pitch_link"/>
-            <origin xyz="${hip_pitch_link_length}  0.0 0.0" rpy="0 0 0" />
+            <origin xyz="${hip_pitch_link_length}  0.0 0.05" rpy="0 0 0" />
             <axis xyz="0 1 0"/>
             <limit velocity="1.0" effort="10" lower="-3.1415" upper="3.1415" />
@@ -32,5 +34,6 @@
             <parent link="${prefix}_hip_pitch_link"/>
             <child link="${prefix}_knee_pitch_link"/>
-            <origin xyz="${knee_pitch_link_length} 0.0 0.0" rpy="0 0 0" />        <axis xyz="0 1 0"/>
+            <origin xyz="${knee_pitch_link_length} 0.0 -0.1" rpy="0 0 0" />
+            <axis xyz="0 1 0"/>
             <limit velocity="1.0" effort="10" lower="-3.1415" upper="3.1415" />
         </joint>
@@ -49,4 +52,14 @@
             <axis xyz="0 0 1"/>
         </joint>
+        <joint name="${prefix}_sole_joint" type="fixed">
+            <parent link="${prefix}_ankle_roll_link"/>
+            <child link="${prefix}_sole"/>
+             <origin xyz="${sole_length} 0.0 0.0" rpy="0 -${pi/2} 0" />
+        </joint>
+        <joint name="${prefix}_toe_joint" type="fixed">
+            <parent link="${prefix}_sole"/>
+            <child link="${prefix}_toe"/>
+             <origin xyz="0.65 ${reflect * 0.1} 0.0" rpy="0 0 0" />
+        </joint>
     </xacro:macro>
 </robot>

File: zeno_description/urdf/zeno_robot.urdf.xacro (robot description, xacro)
@@ -8,9 +8,11 @@
     <xacro:property name="pi" value="3.14159265359" />
     <xacro:property name="shoulder_pitch_angle" value="-0.1418" />
+    <xacro:property name="shoulder_roll_angle" value="0.1418" />
     <xacro:property name="hip_roll_link_length" value="0.148" />
     <xacro:property name="hip_pitch_link_length" value="0.448" />
-    <xacro:property name="knee_pitch_link_length" value="0.7267" />
+    <xacro:property name="knee_pitch_link_length" value="0.6" />
     <xacro:property name="ankle_pitch_link_length" value="0.6846" />
-    <xacro:property name="ankle_roll_link_length" value="0.4622" />
+    <xacro:property name="ankle_roll_link_length" value="0.0" />
+    <xacro:property name="sole_length" value="0.4622" />
     <!-- Head and Torso-->
     <xacro:zeno_head/>
